Commit message: Modified rover schematic

File: pi/ros2_ws/opt/my_robot.urdf (robot description, URDF)
Before this commit: robot my_robot, 6 links, 5 joints
Links:
- removed link caster_wheel
- removed link left_wheel
- removed link right_wheel
- added link back_left_wheel; visual cylinder length=0.05 radius=0.1
- added link back_right_wheel; visual cylinder length=0.05 radius=0.1
- added link front_left_wheel; visual cylinder length=0.05 radius=0.1
- added link front_right_wheel; visual cylinder length=0.05 radius=0.1
Joints:
- removed joint base_caster_wheel_joint
- removed joint base_left_wheel_joint
- removed joint base_right_wheel_joint
- added joint base_back_left_wheel_joint: type fixed, parent base_link, child back_left_wheel, origin xyz=-0.15 0.225 0 rpy=0 0 0, axis 0 1 0
- added joint base_back_right_wheel_joint: type fixed, parent base_link, child back_right_wheel, origin xyz=-0.15 -0.225 0 rpy=0 0 0, axis 0 1 0
- added joint base_front_left_wheel_joint: type fixed, parent base_link, child front_left_wheel, origin xyz=0.15 0.225 0 rpy=0 0 0, axis 0 1 0
- added joint base_front_right_wheel_joint: type fixed, parent base_link, child front_right_wheel, origin xyz=0.15 -0.225 0 rpy=0 0 0, axis 0 1 0

Commit message: Corrected LiDAR angle
LiDAR angular z has been translated in the urdf file by 180 degrees (3.1416 rad)

File: pi/ros2_ws/opt/my_robot.urdf (robot description, URDF)
Before this commit: robot my_robot, 7 links, 6 joints
Joints:
- joint base_laser_joint: origin xyz=0 0 0.225 rpy=0 0 0 -> xyz=0 0 0.225 rpy=0 0 3.1416
